File: Display/Display.kicad_sch (KiCad schematic)
At the start: 505 parts, among them U1 74HC595, U10 74HC595, U11 74HC595, U12 74HC595, U13 74HC595, U14 74HC595, U15 74HC595, U16 74HC595, U17 74HC595, U18 74HC595, U19 74HC595, U2 74HC595, U20 74HC595, U21 74HC595, U22 74HC595, U23 74HC595, U24 74HC595, U25 74HC595, U26 74HC595, U27 74HC595, U28 74HC595, U29 74HC595, U3 74HC595, U30 74HC595, U31 74HC595, U32 74HC595, U33 74HC595, U34 74HC595, U35 74HC595, U36 74HC595, U37 74HC595, U38 74HC595, U39 74HC595, U4 74HC595, U40 74HC595, U41 74HC595, U42 74HC595, U43 74HC595, U44 74HC595, U45 74HC595, U46 74HC595, U47 74HC595, U48 74HC595, U49 74HC595, U5 74HC595, U50 74HC595, U51 74HC595, U52 74HC595, U53 74HC595, U6 74HC595, U7 74HC595, U8 74HC595, U9 74HC595

Commit message: before routing
Parts:
- removed R421, R422, R423, R424: 100, Resistor_SMD:R_0402_1005Metric_Pad0.72x0.64mm_HandSolder, symbol Device:R
- added C1, C10, C11, C12, C13, C14, C15, C16, C17, C18, C19, C2, C20, C21, C22, C23, C24, C25, C26, C27, C28, C29, C3, C30, C31, C32, C33, C34, C35, C36, C37, C38, C39, C4, C40, C41, C42, C43, C44, C45, C46, C47, C48, C49, C5, C50, C51, C52, C53, C6, C7, C8, C9: 100n, Capacitor_SMD:C_0201_0603Metric_Pad0.64x0.40mm_HandSolder, symbol Device:C
- added J1, J4: Conn_01x60, symbol Connector_Generic:Conn_01x60
- added J2, J3: 12402032E202A, External_Parts:CONN_12402032E202A_AMP, symbol External_Parts:12402032E202A
- added S1, S2, S3, S4, S5: TL2230EEF100, External_Parts:SW_TL2230EEF100, symbol External_Parts:TL2230EEF100
Connections:
- net GNDD: now also C1.2, C10.2, C11.2, C12.2, C13.2, C14.2, C15.2, C16.2, C17.2, C18.2, C19.2, C2.2, C20.2, C21.2, C22.2, C23.2, C24.2, C25.2, C26.2, C27.2, C28.2, C29.2, C3.2, C30.2, C31.2, C32.2, C33.2, C34.2, C35.2, C36.2, C37.2, C38.2, C39.2, C4.2, C40.2, C41.2, C42.2, C43.2, C44.2, C45.2, C46.2, C47.2, C48.2, C49.2, C5.2, C50.2, C51.2, C52.2, C53.2, C6.2, C7.2, C8.2, C9.2, J1.49 (Pin_49), J1.51 (Pin_51), J1.53 (Pin_53), J1.55 (Pin_55), J1.57 (Pin_57), J4.1 (Pin_1), J4.13 (Pin_13), J4.17 (Pin_17), J4.21 (Pin_21), J4.25 (Pin_25), J4.29 (Pin_29), J4.33 (Pin_33), J4.37 (Pin_37), J4.41 (Pin_41), J4.5 (Pin_5), J4.50 (Pin_50), J4.52 (Pin_52), J4.54 (Pin_54), J4.56 (Pin_56), J4.58 (Pin_58), J4.60 (Pin_60), J4.9 (Pin_9)
- net RCL: now also J1.56 (Pin_56)
- net SR: now also J1.50 (Pin_50)
- net SRCL: now also J1.52 (Pin_52)
- net SRCR: now also J1.54 (Pin_54)
- net VCC: now also C1.1, C10.1, C11.1, C12.1, C13.1, C14.1, C15.1, C16.1, C17.1, C18.1, C19.1, C2.1, C20.1, C21.1, C22.1, C23.1, C24.1, C25.1, C26.1, C27.1, C28.1, C29.1, C3.1, C30.1, C31.1, C32.1, C33.1, C34.1, C35.1, C36.1, C37.1, C38.1, C39.1, C4.1, C40.1, C41.1, C42.1, C43.1, C44.1, C45.1, C46.1, C47.1, C48.1, C49.1, C5.1, C50.1, C51.1, C52.1, C53.1, C6.1, C7.1, C8.1, C9.1, J1.59 (Pin_59), J1.60 (Pin_60), J4.42 (Pin_42), J4.43 (Pin_43), J4.44 (Pin_44), J4.45 (Pin_45), J4.46 (Pin_46), J4.47 (Pin_47), J4.48 (Pin_48), J4.49 (Pin_49)
- net ~{OE}: now also J1.58 (Pin_58)
- net Misc_QG: now reaches U53.6 (QG)
- net Misc_QG: now also J4.55 (Pin_55)
- net Misc_QE: now reaches U53.4 (QE)
- net Misc_QE: now also J4.59 (Pin_59)
- net Misc_QF: now reaches U53.5 (QF)
- net Misc_QF: now also J4.57 (Pin_57)
- net Misc_QH: now reaches U53.7 (QH)
- net Misc_QH: now also J4.53 (Pin_53)
- net Misc_QH': now reaches U53.9 (QH')
- net Misc_QH': now also J4.51 (Pin_51)
- new net: J4.34 (Pin_34), S5.1
- new net: J4.35 (Pin_35), S5.2
- new net: J4.36 (Pin_36), S5.3
- new net: J4.38 (Pin_38), S5.4
- new net: J4.39 (Pin_39), S5.5
- new net: J4.40 (Pin_40), S5.6
- new net: J4.18 (Pin_18), S3.1
- new net: J4.19 (Pin_19), S3.2
- new net: J4.20 (Pin_20), S3.3
- new net: J4.22 (Pin_22), S3.4
- new net: J4.23 (Pin_23), S3.5
- new net: J4.24 (Pin_24), S3.6
- new net: J1.24 (Pin_24), J2.A1 (GND)
- new net: J1.15 (Pin_15), J2.A10 (RX2-)
- new net: J1.14 (Pin_14), J2.A11 (RX2+)
- new net: J1.13 (Pin_13), J2.A12 (GND)
- new net: J1.23 (Pin_23), J2.A2 (TX1+)
- new net: J1.22 (Pin_22), J2.A3 (TX1-)
- new net: J1.21 (Pin_21), J2.A4 (VBUS)
- new net: J1.20 (Pin_20), J2.A5 (CC1)
- new net: J1.19 (Pin_19), J2.A6 (D+)
- new net: J1.18 (Pin_18), J2.A7 (D-)
- new net: J1.17 (Pin_17), J2.A8 (SBU1)
- new net: J1.16 (Pin_16), J2.A9 (VBUS)
- new net: J1.12 (Pin_12), J2.B1 (GND)
- new net: J1.3 (Pin_3), J2.B10 (RX1-)
- new net: J1.2 (Pin_2), J2.B11 (RX1+)
- new net: J1.1 (Pin_1), J2.B12 (GND)
- new net: J1.11 (Pin_11), J2.B2 (TX2+)
- new net: J1.10 (Pin_10), J2.B3 (TX2-)
- new net: J1.9 (Pin_9), J2.B4 (VBUS)
- new net: J1.8 (Pin_8), J2.B5 (CC1)
- new net: J1.7 (Pin_7), J2.B6 (D+)
- new net: J1.6 (Pin_6), J2.B7 (D-)
- new net: J1.5 (Pin_5), J2.B8 (SBU2)
- new net: J1.4 (Pin_4), J2.B9 (VBUS)
- new net: J4.2 (Pin_2), S1.1
- new net: J4.3 (Pin_3), S1.2
- new net: J4.4 (Pin_4), S1.3
- new net: J4.6 (Pin_6), S1.4
- new net: J4.7 (Pin_7), S1.5
- new net: J4.8 (Pin_8), S1.6
- new net: J1.25 (Pin_25), J3.B12 (GND)
- new net: J1.26 (Pin_26), J3.B11 (RX1+)
- new net: J1.27 (Pin_27), J3.B10 (RX1-)
- new net: J1.28 (Pin_28), J3.B9 (VBUS)
- new net: J1.29 (Pin_29), J3.B8 (SBU2)
- new net: J1.30 (Pin_30), J3.B7 (D-)
- new net: J1.31 (Pin_31), J3.B6 (D+)
- new net: J1.32 (Pin_32), J3.B5 (CC1)
- new net: J1.33 (Pin_33), J3.B4 (VBUS)
- new net: J1.34 (Pin_34), J3.B3 (TX2-)
- new net: J1.35 (Pin_35), J3.B2 (TX2+)
- new net: J1.36 (Pin_36), J3.B1 (GND)
- new net: J1.37 (Pin_37), J3.A12 (GND)
- new net: J1.38 (Pin_38), J3.A11 (RX2+)
- new net: J1.39 (Pin_39), J3.A10 (RX2-)
- new net: J1.40 (Pin_40), J3.A9 (VBUS)
- new net: J1.41 (Pin_41), J3.A8 (SBU1)
- new net: J1.42 (Pin_42), J3.A7 (D-)
- new net: J1.43 (Pin_43), J3.A6 (D+)
- new net: J1.44 (Pin_44), J3.A5 (CC1)
- new net: J1.45 (Pin_45), J3.A4 (VBUS)
- new net: J1.46 (Pin_46), J3.A3 (TX1-)
- new net: J1.47 (Pin_47), J3.A2 (TX1+)
- new net: J1.48 (Pin_48), J3.A1 (GND)
- new net: J4.10 (Pin_10), S2.1
- new net: J4.11 (Pin_11), S2.2
- new net: J4.12 (Pin_12), S2.3
- new net: J4.14 (Pin_14), S2.4
- new net: J4.15 (Pin_15), S2.5
- new net: J4.16 (Pin_16), S2.6
- new net: J4.26 (Pin_26), S4.1
- new net: J4.27 (Pin_27), S4.2
- new net: J4.28 (Pin_28), S4.3
- new net: J4.30 (Pin_30), S4.4
- new net: J4.31 (Pin_31), S4.5
- new net: J4.32 (Pin_32), S4.6
Other:
- moved on the sheet: R1, R10, R100, R101, R102, R103, R104, R105, R106, R107, R108, R109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

Commit message: user save
Parts:
- J1, J4: footprint (none) -> External_Parts:CON_2004850460_MOL
Changed lines of the file:
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@@
 			)
 		)
-		(property "Footprint" ""
+		(property "Footprint" "External_Parts:CON_2004850460_MOL"
 			(at 807.72 458.47 0)
 			(effects
@@
 			)
 		)
-		(property "Footprint" ""
+		(property "Footprint" "External_Parts:CON_2004850460_MOL"
 			(at 101.6 151.13 0)
 			(effects

Commit message: user save
Parts:
- removed C1, C10, C11, C12, C13, C14, C15, C16, C17, C18, C19, C2, C20, C21, C22, C23, C24, C25, C26, C27, C28, C29, C3, C30, C31, C32, C33, C34, C35, C36, C37, C38, C39, C4, C40, C41, C42, C43, C44, C45, C46, C47, C48, C49, C5, C50, C51, C52, C53, C6, C7, C8, C9: 100n, Capacitor_SMD:C_0201_0603Metric_Pad0.64x0.40mm_HandSolder, symbol Device:C
- removed R1, R10, R100, R101, R102, R103, R104, R105, R106, R107, R108, R109, R11, R110, R111, R112, R113, R114, R115, R116, R117, R118, R119, R12, R120, R121, R122, R123, R124, R125, R126, R127, R128, R129, R13, R130, R131, R132, R133, R134, R135, R136, R137, R138, R139, R14, R140, R141, R142, R143, R144, R145, R146, R147, R148, R149, R15, R150, R151, R152, R153, R154, R155, R156, R157, R158, R159, R16, R160, R161, R162, R163, R164, R165, R166, R167, R168, R169, R17, R170, R171, R172, R173, R174, R175, R176, R177, R178, R179, R18, R180, R181, R182, R183, R184, R185, R186, R187, R188, R189, R19, R190, R191, R192, R193, R194, R195, R196, R197, R198, R199, R2, R20, R200, R201, R202, R203, R204, R205, R206, R207, R208, R209, R21, R210, R211, R212, R213, R214, R215, R216, R217, R218, R219, R22, R220, R221, R222, R223, R224, R225, R226, R227, R228, R229, R23, R230, R231, R232, R233, R234, R235, R236, R237, R238, R239, R24, R240, R241, R242, R243, R244, R245, R246, R247, R248, R249, R25, R250, R251, R252, R253, R254, R255, R256, R257, R258, R259, R26, R260, R261, R262, R263, R264, R265, R266, R267, R268, R269, R27, R270, R271, R272, R273, R274, R275, R276, R277, R278, R279, R28, R280, R281, R282, R283, R284, R285, R286, R287, R288, R289, R29, R290, R291, R292, R293, R294, R295, R296, R297, R298, R299, R3, R30, R300, R301, R302, R303, R304, R305, R306, R307, R308, R309, R31, R310, R311, R312, R313, R314, R315, R316, R317, R318, R319, R32, R320, R321, R322, R323, R324, R325, R326, R327, R328, R329, R33, R330, R331, R332, R333, R334, R335, R336, R337, R338, R339, R34, R340, R341, R342, R343, R344, R345, R346, R347, R348, R349, R35, R350, R351, R352, R353, R354, R355, R356, R357, R358, R359, R36, R360, R361, R362, R363, R364, R365, R366, R367, R368, R369, R37, R370, R371, R372, R373, R374, R375, R376, R377, R378, R379, R38, R380, R381, R382, R383, R384, R385, R386, R387, R388, R389, R39, R390, R391, R392, R393, R394, R395, R396, R397, R398, R399, R4, R40, R400, R401, R402, R403, R404, R405, R406, R407, R408, R409, R41, R410, R411, R412, R413, R414, R415, R416, R417, R418, R419, R42, R420, R43, R44, R45, R46, R47, R48, R49, R5, R50, R51, R52, R53, R54, R55, R56, R57, R58, R59, R6, R60, R61, R62, R63, R64, R65, R66, R67, R68, R69, R7, R70, R71, R72, R73, R74, R75, R76, R77, R78, R79, R8, R80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: 100, Resistor_SMD:R_0402_1005Metric_Pad0.72x0.64mm_HandSolder, symbol Device:R
- removed SEGD1, SEGD10, SEGD11, SEGD12, SEGD13, SEGD14, SEGD15, SEGD16, SEGD17, SEGD18, SEGD19, SEGD2, SEGD20, SEGD21, SEGD22, SEGD23, SEGD24, SEGD25, SEGD26, SEGD27, SEGD28, SEGD3, SEGD4, SEGD5, SEGD6, SEGD7, SEGD8, SEGD9: ~, External_Parts:ACPSC04-41SEKWA, symbol External_Parts:ACPSC04-41SEKWA
- removed U1, U10, U11, U12, U13, U14, U15, U16, U17, U18, U19, U2, U20, U21, U22, U23, U24, U25, U26, U27, U28, U29, U3, U30, U31, U32, U33, U34, U35, U36, U37, U38, U39, U4, U40, U41, U42, U43, U44, U45, U46, U47, U48, U49, U5, U50, U51, U52, U53, U6, U7, U8, U9: 74HC595, Package_SO:TSSOP-16_4.4x5mm_P0.65mm, symbol 74xx:74HC595
Connections:
- net Misc_QE is gone; now on net GNDD: J4.59 (Pin_59)
- net Misc_QF is gone; now on net GNDD: J4.57 (Pin_57)
- net Misc_QG is gone; now on net GNDD: J4.55 (Pin_55)
- net Misc_QH is gone; now on net GNDD: J4.53 (Pin_53)
- net Misc_QH' is gone; now on net VCC: J4.51 (Pin_51)
- net GNDD: now also J1.59 (Pin_59), J1.60 (Pin_60); no longer J4.50 (Pin_50)
- net VCC: now also J4.50 (Pin_50); no longer J1.59 (Pin_59), J1.60 (Pin_60)
- no-connect marks 0 -> 1
Other:
- added sheet Digit1 (Digit.kicad_sch)
- added sheet Digit10 (Digit.kicad_sch)
- added sheet Digit11 (Digit.kicad_sch)
- added sheet Digit12 (Digit.kicad_sch)
- added sheet Digit13 (Digit.kicad_sch)
- added sheet Digit14 (Digit.kicad_sch)
- added sheet Digit15 (Digit.kicad_sch)
- added sheet Digit16 (Digit.kicad_sch)
- added sheet Digit17 (Digit.kicad_sch)
- added sheet Digit18 (Digit.kicad_sch)
- added sheet Digit19 (Digit.kicad_sch)
- added sheet Digit2 (Digit.kicad_sch)
- added sheet Digit20 (Digit.kicad_sch)
- added sheet Digit21 (Digit.kicad_sch)
- added sheet Digit22 (Digit.kicad_sch)
- added sheet Digit23 (Digit.kicad_sch)
- added sheet Digit24 (Digit.kicad_sch)
- added sheet Digit25 (Digit.kicad_sch)
- added sheet Digit26 (Digit.kicad_sch)
- added sheet Digit27 (Digit.kicad_sch)
- added sheet Digit28 (Digit.kicad_sch)
- added sheet Digit3 (Digit.kicad_sch)
- added sheet Digit4 (Digit.kicad_sch)
- added sheet Digit5 (Digit.kicad_sch)
- added sheet Digit6 (Digit.kicad_sch)
- added sheet Digit7 (Digit.kicad_sch)
- added sheet Digit8 (Digit.kicad_sch)
- added sheet Digit9 (Digit.kicad_sch)
- moved on the sheet: J1, J2, J3, J4, S1, S2, S3, S4, S5
