File: Display/Display.kicad_sch (KiCad schematic)
At the start: 8 parts, among them J1 Conn_01x60, J2 12402032E202A, J3 12402032E202A

Commit message: Update Display.kicad_sch
Parts:
- S1, S2, S3, S4, S5: value TL2230EEF100 -> TL2285OA; DigiKey Part # (none) -> EG1871-ND
Changed lines of the file:
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@@
 			)
 		)
-		(property "Value" "TL2230EEF100"
+		(property "Value" "TL2285OA"
 			(at 30.48 203.2 0)
 			(effects
@@
 				)
 				(justify bottom)
+				(hide yes)
+			)
+		)
+		(property "DigiKey Part #" "EG1871-ND"
+			(at 30.48 213.36 0)
+			(effects
+				(font
+					(size 1.27 1.27)
+				)
 				(hide yes)
 			)
@@
 			)
 		)
-		(property "Value" "TL2230EEF100"
+		(property "Value" "TL2285OA"
 			(at 30.48 143.51 0)
 			(effects
@@
 				)
 				(justify bottom)
+				(hide yes)
+			)
+		)
+		(property "DigiKey Part #" "EG1871-ND"
+			(at 30.48 153.67 0)
+			(effects
+				(font
+					(size 1.27 1.27)
+				)
 				(hide yes)
 			)
@@
 			)
 		)
-		(property "Value" "TL2230EEF100"
+		(property "Value" "TL2285OA"
 			(at 30.226 156.718 0)
 			(effects
@@
 				)
 				(justify bottom)
+				(hide yes)
+			)
+		)
+		(property "DigiKey Part #" "EG1871-ND"
+			(at 30.48 172.72 0)
+			(effects
+				(font
+					(size 1.27 1.27)
+				)
 				(hide yes)
 			)
@@
 			)
 		)
-		(property "Value" "TL2230EEF100"
+		(property "Value" "TL2285OA"
 			(at 30.48 124.46 0)
 			(effects
@@
 				)
 				(justify bottom)
+				(hide yes)
+			)
+		)
+		(property "DigiKey Part #" "EG1871-ND"
+			(at 30.48 134.62 0)
+			(effects
+				(font
+					(size 1.27 1.27)
+				)
 				(hide yes)
 			)
@@
 			)
 		)
-		(property "Value" "TL2230EEF100"
+		(property "Value" "TL2285OA"
 			(at 30.48 184.15 0)
 			(effects
@@
 				(hide yes)
 			)
+		)
+		(property "DigiKey Part #" "EG1871-ND"
+			(at 30.48 194.31 0)
+			(effects
+				(font
+					(size 1.27 1.27)
+				)
+				(hide yes)
+			)
