File: USB_Audio_EVT/USB_Audio_EVT.kicad_pcb (KiCad board)
At the start: 2 copper layers, 0.6 x 1 mm, 36 parts, among them J101 12402032E202A, J102 Screw_Terminal_01x02, J103 SJ1-3523N, U101 TLV73333PDBV, U102 PCM2706CPJTR, Y101 CSTNE12M0G55A000R0

Commit message: Order V1
Parts:
- moved J102 3.90 mm to (72.5, 60.7), turned to 180 degrees
Connections:
- C101 pad 1: Net-(J102-Pin_2) -> Net-(J102-Pin_1)
- J102 pad 1: GND -> Net-(J102-Pin_1)
- J102 pad 2: Net-(J102-Pin_2) -> GND
- U101 pad 1: Net-(J102-Pin_2) -> Net-(J102-Pin_1)
- U101 pad 3: Net-(J102-Pin_2) -> Net-(J102-Pin_1)
Routing:
- net Net-(J102-Pin_1): track 0.00 -> 18.9 mm
- net Net-(J102-Pin_2): track 17.9 -> 0.00 mm
- net /Previous: track 43.2 -> 45.7 mm
- net /USB_DAC_VDD: track 86.7 -> 87.9 mm
- net GND: vias 0 -> 112
- added copper zone on B.Cu, net GND
- added copper zone on F.Cu, net GND
Other:
- board size 0.6 x 1 mm -> 57.5 x 60 mm
