File: USB_Audio_EVT/USB_Audio_EVT.kicad_sch (KiCad schematic)
At the start: 3 parts, among them J101 12402032E202A, J102 SJ1-3523N, U101 PCM2706CPJTR

Commit message: add some models
Parts:
- added S101: TL2285OA, external_components:SW_TL2230EEF100, symbol external_components:TL2230EEF100
- J101: DigiKey Part # (none) -> 664-12402032E202ACT-ND
- J102: DigiKey Part # (none) -> CP1-3523N-ND
- U101: DigiKey Part # (none) -> 296-40481-1-ND
Changed lines of the file:
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@@
+			)
+		)
+		(property "DigiKey Part #" "296-40481-1-ND"
+			(at 149.86 92.71 0)
+			(effects
+				(font
+					(size 1.27 1.27)
+				)
+				(hide yes)
 			)
 		)
@@
 				(path "/0b97e642-0b10-4a77-9ca5-0c656c23b8f0"
 					(reference "U101")
+					(unit 1)
+				)
+			)
+		)
+	)
+	(symbol
+		(lib_id "external_components:TL2230EEF100")
+		(at 71.12 157.48 0)
+		(unit 1)
+		(exclude_from_sim no)
+		(in_bom yes)
+		(on_board yes)
+		(dnp no)
+		(fields_autoplaced yes)
+		(property "Reference" "S101"
+			(at 71.12 144.78 0)
+			(effects
+				(font
+					(size 1.27 1.27)
+				)
+			)
+		)
+		(property "Value" "TL2285OA"
+			(at 71.12 147.32 0)
+			(effects
+				(font
+					(size 1.27 1.27)
+				)
+			)
+		)
+		(property "Footprint" "external_components:SW_TL2230EEF100"
+			(at 71.12 157.48 0)
+			(effects
+				(font
+					(size 1.27 1.27)
+				)
+				(justify bottom)
+				(hide yes)
+			)
+		)
+		(property "Datasheet" ""
+			(at 71.12 157.48 0)
+			(effects
+				(font
+					(size 1.27 1.27)
+				)
+				(hide yes)
+			)
+		)
+		(property "Description" ""
+			(at 71.12 157.48 0)
+			(effects
+				(font
+					(size 1.27 1.27)
+				)
+				(hide yes)
+			)
+		)
+		(property "PARTREV" "E"
+			(at 71.12 157.48 0)
+			(effects
+				(font
+					(size 1.27 1.27)
+				)
+				(justify bottom)
+				(hide yes)
+			)
+		)
+		(property "STANDARD" "Manufacturer Recommendations"
+			(at 71.12 157.48 0)
+			(effects
+				(font
+					(size 1.27 1.27)
+				)
+				(justify bottom)
+				(hide yes)
+			)
+		)
+		(property "MANUFACTURER" "E-Switch"
+			(at 71.12 157.48 0)
+			(effects
+				(font
+					(size 1.27 1.27)
+				)
+				(justify bottom)
+				(hide yes)
+			)
+		)
+		(property "MAXIMUM_PACKAGE_HEIGHT" "12.5 mm"
+			(at 71.12 157.48 0)
+			(effects
+				(font
+					(size 1.27 1.27)
+				)
+				(justify bottom)
+				(hide yes)
+			)
+		)
+		(property "SNAPEDA_PN" "TL2230EEF140"
+			(at 71.12 157.48 0)
+			(effects
+				(font
+					(size 1.27 1.27)
+				)
+				(justify bottom)
+				(hide yes)
+			)
+		)
+		(property "DigiKey Part #" "EG1871-ND"
+			(at 71.12 157.48 0)
+			(effects
+				(font
+					(size 1.27 1.27)
+				)
+				(hide yes)
+			)
+		)
+		(pin "1"
+		)
+		(pin "3"
+		)
+		(pin "4"
+		)
+		(pin "6"
+		)
+		(pin "2"
+		)
+		(pin "5"
+		)
+		(instances
+			(project ""
+				(path "/0b97e642-0b10-4a77-9ca5-0c656c23b8f0"
+					(reference "S101")
 					(unit 1)
 				)
@@
 			)
 		)
+		(property "DigiKey Part #" "CP1-3523N-ND"
+			(at 121.92 181.61 0)
+			(effects
+				(font
+					(size 1.27 1.27)
+				)
+				(hide yes)
+			)
+		)
 		(pin "2"
 		)
@@
 			(at 46.99 137.16 0)
 			(effects
+				(font
+					(size 1.27 1.27)
+				)
+				(hide yes)
+			)
+		)
+		(property "DigiKey Part #" "664-12402032E202ACT-ND"
+			(at 46.99 137.16 0)
+			(effects

Commit message: add more components
Parts:
- added C101: 100u, Capacitor_Tantalum_SMD:CP_EIA-3528-21_Kemet-B_HandSolder, symbol Device:C_Polarized
- added C102: 22n, Capacitor_SMD:C_0603_1608Metric_Pad1.08x0.95mm_HandSolder, symbol Device:C
- added C215: 10u, Capacitor_SMD:C_0805_2012Metric_Pad1.18x1.45mm_HandSolder, symbol Device:C
- added C501: 1u, Capacitor_SMD:C_0603_1608Metric_Pad1.08x0.95mm_HandSolder, symbol Device:C
- added R101: 1k5, Resistor_SMD:R_0402_1005Metric_Pad0.72x0.64mm_HandSolder, symbol Device:R
- added R102: 3k3, Resistor_SMD:R_0402_1005Metric_Pad0.72x0.64mm_HandSolder, symbol Device:R
- added R103: 22, Resistor_SMD:R_0402_1005Metric_Pad0.72x0.64mm_HandSolder, symbol Device:R
- added R104: 16, Resistor_SMD:R_0402_1005Metric_Pad0.72x0.64mm_HandSolder, symbol Device:R
- added R105: 1M, Resistor_SMD:R_0402_1005Metric_Pad0.72x0.64mm_HandSolder, symbol Device:R
- added Y101: CSTNE12M0G55A000R0, external_components:OSC_CSTNE12M0G55A000R0, symbol external_components:CSTNE12M0G55A000R0

Commit message: some routing
Parts:
- removed C215: 10u, Capacitor_SMD:C_0805_2012Metric_Pad1.18x1.45mm_HandSolder, symbol Device:C
- added C101, C102, C107: 10u, Capacitor_SMD:C_0805_2012Metric_Pad1.18x1.45mm_HandSolder, symbol Device:C
- added C103: 22n, Capacitor_SMD:C_0603_1608Metric_Pad1.08x0.95mm_HandSolder, symbol Device:C
- added C105, C109, C110, C112: 1u, Capacitor_SMD:C_0603_1608Metric_Pad1.08x0.95mm_HandSolder, symbol Device:C
- added C106: 100u, Capacitor_Tantalum_SMD:CP_EIA-3528-21_Kemet-B_HandSolder, symbol Device:C_Polarized
- added J102: Screw_Terminal_01x02, TerminalBlock_Phoenix:TerminalBlock_Phoenix_MKDS-1,5-2-5.08_1x02_P5.08mm_Horizontal, symbol Connector:Screw_Terminal_01x02
- added R101, R103: 5k1, Resistor_SMD:R_0402_1005Metric_Pad0.72x0.64mm_HandSolder, symbol Device:R
- added R102: 1k5, Resistor_SMD:R_0402_1005Metric_Pad0.72x0.64mm_HandSolder, symbol Device:R
- added R105: 22, Resistor_SMD:R_0402_1005Metric_Pad0.72x0.64mm_HandSolder, symbol Device:R
- added R107: 16, Resistor_SMD:R_0402_1005Metric_Pad0.72x0.64mm_HandSolder, symbol Device:R
- added R109, R110, R111: 3k3, Resistor_SMD:R_0402_1005Metric_Pad0.72x0.64mm_HandSolder, symbol Device:R
- added S102, S103, S104, S105: TL2285OA, external_components:SW_TL2230EEF100, symbol external_components:TL2230EEF100
- added U101: TLV73333PDBV, Package_TO_SOT_SMD:SOT-23-5, symbol Regulator_Linear:TLV73333PDBV
- renumbered C102 to C104, C101 to C108, C501 to C111, J102 to J103, R103 to R104, R101 to R106, R104 to R108, R102 to R112, R105 to R113, U101 to U102
Connections:
- net at R108.1: now also C104.2
- net GND: now reaches R108.2
- net GND: now also C111.2, J101.A1 (GND), J101.A12 (GND), J101.B1 (GND), J101.B12 (GND), J103.1, R112.2, U102.1 (PGND), U102.20 (DGND), U102.25 (ZGND), U102.26 (AGNDL), U102.3 (HOST), U102.31 (AGNDR), Y101.2, C101.2, C102.2, C105.2, C107.2, C109.2, C110.2, C112.2, J102.1 (Pin_1), R101.2, R103.2, R107.2, R109.2, R110.2, R111.2, U101.2 (GND)
- net at C104.1: now also C108.1, U102.28 (VOUTL), R110.1
- net at C111.1: now also U102.27 (VCCL)
- net USB_DAC_OUT_L: now reaches C108.2
- net USB_DAC_OUT_L: now also J103.2, R112.1
- net USB_DAC_XT1: now reaches Y101.1
- net USB_DAC_XT1: now also R113.1, U102.12 (XTI)
- net USB_DAC_XT0: now reaches Y101.3
- net USB_DAC_XT0: now also R113.2, U102.13 (XTO)
- net at R106.1: now also U102.15 (DT)
- net USB_DAC_VDD: now reaches R106.2
- net USB_DAC_VDD: now also U102.10 (TEST), U102.16 (PSEL), U102.9 (FSEL), C102.1, R102.1, U101.5 (OUT)
- net DAC_D+: now reaches R104.1
- net DAC_D+: now also J101.A6 (D+), J101.B6 (D+), R102.2
- net at R104.2: now also U102.23 (D+)
- net ~{USB_DAC_SSPND}: now reaches U102.11 (~{SSPND})
- net ~{USB_DAC_SSPND}: now also S101.2, S102.2, S103.2, S104.2, S105.2
- net Previous: now reaches U102.19 (FUNC1)
- net Previous: now also S103.3
- net at U102.2 (VCCP): now also C110.1
- net at U102.21 (VDD): now also C105.1
- net at U102.22 (D-): now also R105.2
- net DAC_VBUS: now reaches U102.24 (VBUS)
- net DAC_VBUS: now also J101.A4 (VBUS), J101.A9 (VBUS), J101.B4 (VBUS), J101.B9 (VBUS), C112.1
- net at U102.29 (VOUTR): now also C103.1, C106.1, R109.1
- net at U102.30 (VCCR): now also C109.1
- net at U102.32 (VCOM): now also C107.1
- net Play/Pause: now reaches U102.4 (FUNC3)
- net Play/Pause: now also S101.3
- net Next: now reaches U102.5 (FUNC0)
- net Next: now also S102.3
- net VOL+: now reaches U102.7 (HID1/MC)
- net VOL+: now also S104.3
- net VOL-: now reaches U102.8 (HID2/MD)
- net VOL-: now also S105.3
- net USB_DAC_OUT_R: now reaches J103.3
- net USB_DAC_OUT_R: now also C106.2, R111.1
- net DAC_CC1: now reaches J101.A5 (CC1)
- net DAC_CC1: now also R101.1
- net DAC_D-: now reaches J101.A7 (D-)
- net DAC_D-: now also J101.B7 (D-), R105.1
- net DAC_CC2: now reaches J101.B5 (CC1)
- net DAC_CC2: now also R103.1
- new net: C103.2, R107.1
- new net: C101.1, J102.2 (Pin_2), U101.1 (IN), U101.3 (EN)
- no-connect marks 0 -> 14
Other:
- moved on the sheet: C104, C108, C111, J101, J103, R104, R106, R108, R112, R113, S101, Y101

Commit message: Order V1
Connections:
- net GND: now also J102.2 (Pin_2); no longer J102.1 (Pin_1)
- net at C101.1, U101.1 (IN), U101.3 (EN): now also J102.1 (Pin_1); no longer J102.2 (Pin_2)
Other:
- moved on the sheet: J102
Changed lines of the file:
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@@
 	(symbol
 		(lib_id "Connector:Screw_Terminal_01x02")
-		(at 34.29 30.48 180)
+		(at 34.29 27.94 0)
+		(mirror y)
 		(unit 1)
 		(exclude_from_sim no)
@@
 		(on_board yes)
 		(dnp no)
-		(fields_autoplaced yes)
 		(property "Reference" "J102"
-			(at 34.29 21.59 0)
+			(at 34.29 22.606 0)
 			(effects
 				(font
@@
 		)
 		(property "Value" "Screw_Terminal_01x02"
-			(at 34.29 24.13 0)
+			(at 34.29 24.892 0)
 			(effects
 				(font
@@
 		)
 		(property "Footprint" "TerminalBlock_Phoenix:TerminalBlock_Phoenix_MKDS-1,5-2-5.08_1x02_P5.08mm_Horizontal"
-			(at 34.29 30.48 0)
+			(at 34.29 27.94 0)
 			(effects
 				(font
@@
 		)
 		(property "Datasheet" "~"
-			(at 34.29 30.48 0)
+			(at 34.29 27.94 0)
 			(effects
 				(font
@@
 		)
 		(property "Description" "Generic screw terminal, single row, 01x02, script generated (kicad-library-utils/schlib/autogen/connector/)"
-			(at 34.29 30.48 0)
+			(at 34.29 27.94 0)
 			(effects
 				(font
