File: Systemboard/Systemboard.kicad_sch (KiCad schematic)
At the start: 7 parts, among them J1 Conn_01x60, J108 Prog BT, U101 ESP32-WROOM-32E

Commit message: user save
Parts:
- added C216: 100n, Capacitor_SMD:C_0805_2012Metric_Pad1.18x1.45mm_HandSolder, symbol Device:C
- added C217: 10u, Capacitor_SMD:C_0805_2012Metric_Pad1.18x1.45mm_HandSolder, symbol Device:C
Connections:
- net +3V3: now also U101.2 (VDD), C216.1, C217.2
- net GND: now also C216.2, C217.1
Other:
- added sheet Power Supply (Power_Supply.kicad_sch)

Commit message: user save
Other:
- sheet Shunt renamed USB Charger
- sheet USB Charger ports: added CC1, CC2, V_CHARGER; removed Vin-
- note added: "check for linear voltage regulator on jlc display illumination by using an optoelectric feedback with a vreg reed switches"
- note removed: "check whether the headset uses NC or NO switches and reserve that switches for them amplifier power supply high-current 5V, +/-12V maybe, high-current dimmable 2V-3V3 reed switches amp input mux"
Changed lines of the file:
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@@
 	(generator_version "10.0")
 	(paper "A4")
-	(text "check whether the headset uses NC or NO switches and reserve that switches for them\n\namplifier\n\npower supply\nhigh-current 5V, +/-12V maybe, high-current dimmable 2V-3V3\n\nreed switches\namp input mux"
+	(text "check for linear voltage regulator on jlc\n\ndisplay illumination by using an optoelectric feedback with a vreg\n\nreed switches"
 		(exclude_from_sim no)
 		(at 84.836 22.352 0)
@@
 	(wire
 		(pts
-			(xy 241.3 130.81) (xy 243.84 130.81)
+			(xy 208.28 144.78) (xy 205.74 144.78)
 		)
 		(stroke
@@
 	(wire
 		(pts
-			(xy 208.28 144.78) (xy 205.74 144.78)
+			(xy 138.43 66.04) (xy 139.7 66.04)
 		)
 		(stroke
@@
 	(wire
 		(pts
-			(xy 138.43 66.04) (xy 139.7 66.04)
+			(xy 193.04 64.77) (xy 196.85 64.77)
 		)
 		(stroke
@@
 	(wire
 		(pts
-			(xy 193.04 64.77) (xy 196.85 64.77)
+			(xy 96.52 162.56) (xy 130.81 162.56)
 		)
 		(stroke
@@
 	(wire
 		(pts
-			(xy 96.52 162.56) (xy 130.81 162.56)
+			(xy 31.75 77.47) (xy 40.64 77.47)
 		)
 		(stroke
@@
 	(wire
 		(pts
-			(xy 31.75 77.47) (xy 40.64 77.47)
+			(xy 242.57 140.97) (xy 243.84 140.97)
 		)
 		(stroke
@@
 	(wire
 		(pts
+			(xy 242.57 137.16) (xy 243.84 137.16)
+		)
+		(stroke
+			(width 0)
+			(type default)
+		)
+	)
+	(wire
+		(pts
 			(xy 186.69 92.71) (xy 191.77 92.71)
 		)
@@
 		)
 	)
+	(wire
+		(pts
+			(xy 242.57 130.81) (xy 243.84 130.81)
+		)
+		(stroke
+			(width 0)
+			(type default)
+		)
+	)
 	(label "BTN_1_COM_B"
 		(at 124.46 20.32 180)
@@
 		)
 	)
+	(label "CHARGER_CC2"
+		(at 242.57 140.97 180)
+		(effects
+			(font
+				(size 1.27 1.27)
+			)
+			(justify right bottom)
+		)
+	)
 	(label "CHARGER_D-"
 		(at 31.75 59.69 0)
@@
 	)
 	(label "CHARGER_VBUS"
-		(at 241.3 130.81 180)
+		(at 242.57 130.81 180)
 		(effects
 			(font
@@
 		)
 	)
+	(label "CHARGER_CC1"
+		(at 242.57 137.16 180)
+		(effects
+			(font
+				(size 1.27 1.27)
+			)
+			(justify right bottom)
+		)
+	)
 	(label "DAC_CC1"
 		(at 31.75 26.67 0)
@@
 	(sheet
 		(at 243.84 110.49)
-		(size 25.4 25.4)
+		(size 25.4 34.29)
 		(exclude_from_sim no)
 		(in_bom yes)
@@
 			(color 0 0 0 0)
 		)
-		(property "Sheetname" "Shunt"
+		(property "Sheetname" "USB Charger"
 			(at 243.84 109.7784 0)
 			(show_name no)
@@
 		)
 		(property "Sheetfile" "Shunt.kicad_sch"
-			(at 243.84 136.4746 0)
+			(at 243.84 145.3646 0)
 			(show_name no)
 			(do_not_autoplace no)
@@
 			)
 		)
-		(pin "Vin-" passive
+		(pin "V_CHARGER" passive
 			(at 243.84 130.81 180)
 			(effects
 				(font
+					(size 1.27 1.27)
+				)
+				(justify left)
+			)
+		)
+		(pin "CC2" output
+			(at 243.84 140.97 180)
+			(effects
+				(font
+					(size 1.27 1.27)
+				)
+				(justify left)
+			)
+		)
+		(pin "CC1" output
+			(at 243.84 137.16 180)
+			(effects
+				(font

Commit message: user save
Parts:
- added J2: Conn_01x02, Connector_Wire:SolderWire-1sqmm_1x02_P5.4mm_D1.4mm_OD2.7mm, symbol Connector_Generic:Conn_01x02
- added J3, J4: Conn_01x01, Connector_Wire:SolderWire-2.5sqmm_1x01_D2.4mm_OD3.6mm, symbol Connector_Generic:Conn_01x01
- added R136: 3k3, Resistor_SMD:R_0402_1005Metric_Pad0.72x0.64mm_HandSolder, symbol Device:R
- added R143: 10k, Resistor_SMD:R_0402_1005Metric_Pad0.72x0.64mm_HandSolder, symbol Device:R
- added Speaker_Front, Speaker_Rear: Conn_02x02_Odd_Even, Connector_Wire:SolderWire-1sqmm_1x04_P5.4mm_D1.4mm_OD2.7mm, symbol Connector_Generic:Conn_02x02_Odd_Even
Connections:
- net GND: now also J4.1 (Pin_1), R136.2
- net Dimm_Display: now reaches U101.23 (IO15)
- net at U101.26 (IO4): now also R136.1, R143.1
- new net +Acc: J2.1 (Pin_1)
- new net +B: J3.1 (Pin_1)
- new net Illumination: J2.2 (Pin_2), R143.2
- new net Speaker_NL: Speaker_Front.2 (Pin_2), Speaker_Rear.2 (Pin_2)
- new net Speaker_NR: Speaker_Front.4 (Pin_4), Speaker_Rear.4 (Pin_4)
- new net Speaker_PL: Speaker_Front.1 (Pin_1), Speaker_Rear.1 (Pin_1)
- new net Speaker_PR: Speaker_Front.3 (Pin_3), Speaker_Rear.3 (Pin_3)
Other:
- sheet Power Supply ports: added Acc+, B+, Dimming, V_Display; removed none

Commit message: user save
Connections:
- net ~{AMP_FAIL}: now reaches U101.27 (IO16)
- net ~{BT}/USB: now reaches U101.28 (IO17)
- net EN renamed ESP_EN
- net IO0_BT renamed ESP_IO0
- net MUTE renamed SPEAKER_EN
- net RCL renamed Display_RCL
- net RXD_BT renamed ESP_RXD
- net SR renamed Display_SR
- net SRCL renamed Display_SRCL
- net TXD_BT renamed ESP_TXD
- net USB_SHUNT_SCL renamed CHARGER_SHUNT_SCL
- net USB_SHUNT_SDA renamed CHARGER_SHUNT_SDA
Other:
- sheet Amplifier ports: added ~{Error}, ~{Mute}; removed Mute
- note added: "reed switches"
- note removed: "check for linear voltage regulator on jlc display illumination by using an optoelectric feedback with a vreg reed switches"

Commit message: user save
Connections:
- net SPEAKER_EN: no longer U101.24 (IO2)
- net USB_DAC_EN: no longer U101.16 (IO13)
- net ~{BT}/USB: no longer U101.28 (IO17)
- new net CONFIG_SCL: U101.28 (IO17)
- new net CONFIG_SDA: U101.24 (IO2)
- new net CONFIG_Update: U101.16 (IO13)
Other:
- added sheet Configurator (Configurator.kicad_sch)
- sheet Power Supply ports: added +5V_On, Display_On; removed none

Commit message: user save
Parts:
- added J5: PTV112-4420A-A503, External_Parts:CONN_A503, symbol External_Parts:PTV112-4420A-A503
Connections:
- net Amplifier Input Mux/AMPLIFIER_IN_L: now also J5.6 (3)
- net Amplifier Input Mux/AMPLIFIER_IN_R: now also J5.5 (3)
- net GND: now also J5.2 (1), J5.3 (1)
- new net Amplifier/Amplifier_In_L: J5.1 (2)
- new net Amplifier/Amplifier_In_R: J5.4 (2)
Other:
- moved on the sheet: C216, C217, J2, J3, J4, R103, R136, R143, Speaker_Front, Speaker_Rear, U101

Commit message: add switch
Parts:
- added R150, R152: 10k, Resistor_SMD:R_0402_1005Metric_Pad0.72x0.64mm_HandSolder, symbol Device:R
- added R151, R153: 47, Resistor_SMD:R_0603_1608Metric_Pad0.98x0.95mm_HandSolder, symbol Device:R
- added S1, S2: SS0750301F040P1A, External_Parts:SS0750301F040P1A, symbol External_Parts:SS0750301F040P1A
Connections:
- net +3V3: now also R150.2, R152.2
- net GND: now also S1.1 (C), S2.1 (C)
- net at U101.4 (SENSOR_VP): now also R151.1
- net at U101.5 (SENSOR_VN): now also R153.1
- new net: R150.1, R151.2, S1.2 (NO)
- new net: R152.1, R153.2, S2.2 (NO)
- no-connect marks 2 -> 0
Other:
- moved on the sheet: C101, C216, C217, J1, J108, J2, J3, J4, J5, R101, R103, R117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

Commit message: user save part number
Parts:
- J108: DigiKey Part # (none) -> S7004-ND
- S1, S2: DigiKey Part # (none) -> EG4924-ND
- U101: JLCPCB Part # (none) -> C701343
