File: Systemboard/Amplifier.kicad_sch (KiCad schematic)
At the start: 19 parts, among them Q501 MMBT3904, U501 TPA3118D2DAPR

Commit message: Add Amp
Parts:
- removed C506: 1n, Capacitor_SMD:C_0603_1608Metric_Pad1.08x0.95mm_HandSolder, symbol Device:C
- removed C507: 10n, Capacitor_SMD:C_0603_1608Metric_Pad1.08x0.95mm_HandSolder, symbol Device:C
- removed C508: 220n, Resistor_SMD:R_0805_2012Metric_Pad1.20x1.40mm_HandSolder, symbol Device:C
- removed R507: 3R3, Resistor_SMD:R_0805_2012Metric_Pad1.20x1.40mm_HandSolder, symbol Device:R
- added C1, C19, C22: 100n, Capacitor_SMD:C_0805_2012Metric_Pad1.18x1.45mm_HandSolder, symbol Device:C
- added C10, C11, C12, C13, C20, C21: 1n, Capacitor_SMD:C_0603_1608Metric_Pad1.08x0.95mm_HandSolder, symbol Device:C
- added C14, C15, C16, C17, C2: 10n, Capacitor_SMD:C_0603_1608Metric_Pad1.08x0.95mm_HandSolder, symbol Device:C
- added C18, C23: 220u, External_Parts:CAP_EEHZU1H221P, symbol Device:C_Polarized
- added C3, C4, C5, C6: 220n, Resistor_SMD:R_0805_2012Metric_Pad1.20x1.40mm_HandSolder, symbol Device:C
- added C7, C8, C9: 680n, Resistor_SMD:R_0805_2012Metric_Pad1.20x1.40mm_HandSolder, symbol Device:C
- added L1, L2, L3: 10u, External_Parts:IND_VLS6045EX-100M, symbol Device:L
- added R2, R3, R4, R5, R6: 3R3, Resistor_SMD:R_0805_2012Metric_Pad1.20x1.40mm_HandSolder, symbol Device:R
- L501: value L -> 10u
Connections:
- net +12V is gone; now on net PVCC: R503.1, R504.1
- net GND: now also C509.2, C1.2, C10.2, C11.2, C12.2, C13.2, C14.2, C15.2, C16.2, C17.2, C18.2, C19.2, C2.2, C20.2, C21.2, C22.2, C23.2, C7.2, C8.2, C9.2
- net PVCC: now also U501.17 (AVCC), C18.1, C19.1, C2.1, C20.1, C21.1, C22.1, C23.1, R2.1
- net at U501.20 (BSNL): now also C6.1
- net at U501.21 (OUTNL): now also L501.1, C6.2
- net at U501.23 (OUTPL): now also C4.2, L2.1
- net at U501.24 (BSPL): now also C4.1
- net at U501.26 (BSNR): now also C5.1
- net at U501.27 (OUTNR): now also C5.2, L1.1
- net at U501.29 (OUTPR): now also C3.2, L3.1
- net at U501.30 (BSPR): now also C3.1
- net Amplifier_Out_NL: now reaches L501.2
- net Amplifier_Out_NL: now also C509.1, C10.1, R3.1
- new net: C17.1, R6.2
- new net: C15.1, R4.2
- new net: C1.1, R2.2
- new net: C14.1, R3.2
- new net: C16.1, R5.2
- new net Amplifier_Out_NR: C11.1, C7.1, L1.2, R4.1
- new net Amplifier_Out_PL: C12.1, C8.1, L2.2, R5.1
- new net Amplifier_Out_PR: C13.1, C9.1, L3.2, R6.1
Other:
- moved on the sheet: C501, C502, C503, C504, C505, C509, L501, Q501, R501, R502, R503, R504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

Commit message: add jlc part numbers
Parts:
- C1, C19, C22: JLCPCB Part # (none) -> C28233
- C10, C11, C12, C13, C20, C21: JLCPCB Part # (none) -> C1588
- C14, C15, C16, C17, C2: JLCPCB Part # (none) -> C57112
- C3, C4, C5, C6: JLCPCB Part # (none) -> C5378
- C501, C502, C503, C504, C505: JLCPCB Part # (none) -> C15849
- R501, R503, R504, R506: JLCPCB Part # (none) -> C25803

Commit message: add more components
Parts:
- R502, R505: JLCPCB Part # (none) -> C4184
Changed lines of the file:
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@@
 			)
 		)
-		(property "JLCPCB Part #" ""
+		(property "JLCPCB Part #" "C4184"
 			(at 59.69 110.49 90)
 			(effects
@@
 			)
 		)
-		(property "JLCPCB Part #" ""
+		(property "JLCPCB Part #" "C4184"
 			(at 156.21 148.59 0)
 			(effects

Commit message: KiCad 10
Parts:
- U501: DESCRIPTION Audio Amp Speaker 1-CH Mono/2-CH Stereo 50W Class-D 32-Pin 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 -> (none)

Commit message: user save
Parts:
- removed Q501: MMBT3904, Package_TO_SOT_SMD:SOT-23, symbol Transistor_BJT:MMBT3904
- removed R505: 20k, Resistor_SMD:R_0603_1608Metric_Pad0.98x0.95mm_HandSolder, symbol Device:R
- removed R506: 100k, Resistor_SMD:R_0603_1608Metric_Pad0.98x0.95mm_HandSolder, symbol Device:R
- added Q2: MMBT5551L, Package_TO_SOT_SMD:SOT-23, symbol Transistor_BJT:MMBT5551L
- added R135: 3k3, Resistor_SMD:R_0402_1005Metric_Pad0.72x0.64mm_HandSolder, symbol Device:R
Connections:
- net GND: now also Q2.2 (E)
- net Mute: now also R135.1
- net at R503.2, U501.12 (MUTE): now also Q2.3 (C)
- net PVCC renamed +12V
- new net: Q2.1 (B), R135.2

Commit message: user save
Parts:
- added R144: 10k, Resistor_SMD:R_0402_1005Metric_Pad0.72x0.64mm_HandSolder, symbol Device:R
- added R145: 3k3, Resistor_SMD:R_0402_1005Metric_Pad0.72x0.64mm_HandSolder, symbol Device:R
Connections:
- net GND: now also R145.2
- net at R504.2, U501.2 (SDZ), U501.3 (FAULTZ): now also R144.2
- net Mute renamed ~{Mute}
- new net ~{Error}: R144.1, R145.1

Commit message: user save part number
Parts:
- L1, L2, L3, L501: JLCPCB Part # (none) -> C168076
- Q2: JLCPCB Part # (none) -> C2145
- R2, R3, R4, R5, R6: JLCPCB Part # (none) -> C16257
- U501: JLCPCB Part # (none) -> C46497
