File: Systemboard/Amplifier.kicad_sch (KiCad schematic)
At the start: 47 parts, among them Q2 MMBT5551L, U501 TPA3118D2DAPR

Commit message: update component numbers
Parts:
- removed C18, C23: 220u, External_Parts:CAP_EEHZU1H221P, symbol Device:C_Polarized
- added C34, C35: 220µ, Capacitor_THT:CP_Radial_D6.3mm_P2.50mm, symbol Device:C_Polarized
- C509, C7, C8, C9: footprint Resistor_SMD:R_0805_2012Metric_Pad1.20x1.40mm_HandSolder -> Capacitor_SMD:C_1206_3216Metric_Pad1.33x1.80mm_HandSolder; DigiKey Part # 1276-7009-1-ND -> (none); JLCPCB Part # (none) -> C1881
Connections:
- net +12V: now also C34.1, C35.1
- net GND: now also C34.2, C35.2
