File: Systemboard/Configurator.kicad_sch (KiCad schematic)
At the start: 2 parts, among them U10 74HC595

Commit message: prep board
Connections:
- no-connect marks 1 -> 4
Changed lines of the file:
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@@
+	)
+	(no_connect
+		(at 149.86 97.79)
+	)
+	(no_connect
+		(at 149.86 102.87)
+	)
+	(no_connect
+		(at 149.86 100.33)
 	)
 	(no_connect
