File: Systemboard/Debouncer.kicad_sch (KiCad schematic)
At the start: 19 parts, among them U102 74HC14, U401 74HC14

Commit message: add jlc part numbers
Parts:
- C102, C103, C104, C105, C106, C401: JLCPCB Part # (none) -> C28233
- R102, R106, R108, R110, R112: footprint Resistor_SMD:R_0402_1005Metric_Pad0.72x0.64mm_HandSolder -> Resistor_SMD:R_0603_1608Metric_Pad0.98x0.95mm_HandSolder; DigiKey Part # P47DCCT-ND -> 311-47.0HRCT-ND; JLCPCB Part # (none) -> C23182
- R104, R105, R107, R109, R111, R113: JLCPCB Part # (none) -> C25744
Changed lines of the file:
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@@
+			)
+		)
+		(property "JLCPCB Part #" ""
+			(at 127 146.05 0)
+			(effects
+				(font
+					(size 1.27 1.27)
+				)
+				(hide yes)
 			)
 		)
@@
 			)
 		)
-		(property "Footprint" "Resistor_SMD:R_0402_1005Metric_Pad0.72x0.64mm_HandSolder"
+		(property "Footprint" "Resistor_SMD:R_0603_1608Metric_Pad0.98x0.95mm_HandSolder"
 			(at 156.21 127.762 90)
 			(effects
@@
 			)
 		)
-		(property "DigiKey Part #" "P47DCCT-ND"
+		(property "DigiKey Part #" "311-47.0HRCT-ND"
+			(at 156.21 129.54 90)
+			(effects
+				(font
+					(size 1.27 1.27)
+				)
+				(hide yes)
+			)
+		)
+		(property "JLCPCB Part #" "C23182"
 			(at 156.21 129.54 90)
 			(effects
@@
 		)
 		(property "DigiKey Part #" "1276-1003-1-ND"
+			(at 166.37 85.09 0)
+			(effects
+				(font
+					(size 1.27 1.27)
+				)
+				(hide yes)
+			)
+		)
+		(property "JLCPCB Part #" "C28233"
 			(at 166.37 85.09 0)
 			(effects
@@
 			)
 		)
-		(property "Footprint" "Resistor_SMD:R_0402_1005Metric_Pad0.72x0.64mm_HandSolder"
+		(property "Footprint" "Resistor_SMD:R_0603_1608Metric_Pad0.98x0.95mm_HandSolder"
 			(at 179.07 78.232 90)
 			(effects
@@
 			)
 		)
-		(property "DigiKey Part #" "P47DCCT-ND"
+		(property "DigiKey Part #" "311-47.0HRCT-ND"
+			(at 179.07 80.01 90)
+			(effects
+				(font
+					(size 1.27 1.27)
+				)
+				(hide yes)
+			)
+		)
+		(property "JLCPCB Part #" "C23182"
 			(at 179.07 80.01 90)
 			(effects
@@
 			)
 		)
+		(property "JLCPCB Part #" ""
+			(at 127 80.01 0)
+			(effects
+				(font
+					(size 1.27 1.27)
+				)
+				(hide yes)
+			)
+		)
 		(pin "1"
 		)
@@
 			)
 		)
+		(property "JLCPCB Part #" "C25744"
+			(at 143.51 90.17 0)
+			(effects
+				(font
+					(size 1.27 1.27)
+				)
+				(hide yes)
+			)
+		)
 		(pin "1"
 		)
@@
 		)
 		(property "DigiKey Part #" "1276-3431-1-ND"
+			(at 143.51 57.15 0)
+			(effects
+				(font
+					(size 1.27 1.27)
+				)
+				(hide yes)
+			)
+		)
+		(property "JLCPCB Part #" "C25744"
 			(at 143.51 57.15 0)
 			(effects
@@
 			)
 		)
+		(property "JLCPCB Part #" "C28233"
+			(at 166.37 118.11 0)
+			(effects
+				(font
+					(size 1.27 1.27)
+				)
+				(hide yes)
+			)
+		)
 		(pin "2"
 		)
@@
 			)
 		)
-		(property "Footprint" "Resistor_SMD:R_0402_1005Metric_Pad0.72x0.64mm_HandSolder"
+		(property "Footprint" "Resistor_SMD:R_0603_1608Metric_Pad0.98x0.95mm_HandSolder"
 			(at 179.07 111.252 90)
 			(effects
@@
 			)
 		)
-		(property "DigiKey Part #" "P47DCCT-ND"
+		(property "DigiKey Part #" "311-47.0HRCT-ND"
+			(at 179.07 113.03 90)
+			(effects
+				(font
+					(size 1.27 1.27)
+				)
+				(hide yes)
+			)
+		)
+		(property "JLCPCB Part #" "C23182"
 			(at 179.07 113.03 90)
 			(effects
@@
 		)
 		(property "DigiKey Part #" "1276-1003-1-ND"
+			(at 54.61 40.64 0)
+			(effects
+				(font
+					(size 1.27 1.27)
+				)
+				(hide yes)
+			)
+		)
+		(property "JLCPCB Part #" "C28233"
 			(at 54.61 40.64 0)
 			(effects
@@
 			)
 		)
+		(property "JLCPCB Part #" ""
+			(at 127 63.5 0)
+			(effects
+				(font
+					(size 1.27 1.27)
+				)
+				(hide yes)
+			)
+		)
 		(pin "1"
 		)
@@
 			)
 		)
+		(property "JLCPCB Part #" ""
+			(at 127 96.52 0)
+			(effects
+				(font
+					(size 1.27 1.27)
+				)
+				(hide yes)
+			)
+		)
 		(pin "1"
 		)
@@
 			)
 		)
+		(property "JLCPCB Part #" ""
+			(at 127 129.54 0)
+			(effects
+				(font
+					(size 1.27 1.27)
+				)
+				(hide yes)
+			)
+		)
 		(pin "1"
 		)
@@
 			)
 		)
+		(property "JLCPCB Part #" "C25744"
+			(at 166.37 106.68 0)
+			(effects
+				(font
+					(size 1.27 1.27)
+				)
+				(hide yes)
+			)
+		)
 		(pin "1"
 		)
@@
 			)
 		)
+		(property "JLCPCB Part #" "C28233"
+			(at 143.51 68.58 0)
+			(effects
+				(font
+					(size 1.27 1.27)
+				)
+				(hide yes)
+			)
+		)
 		(pin "2"
 		)
@@
 		)
 		(property "DigiKey Part #" "1276-3431-1-ND"
+			(at 166.37 73.66 0)
+			(effects
+				(font
+					(size 1.27 1.27)
+				)
+				(hide yes)
+			)
+		)
+		(property "JLCPCB Part #" "C25744"
 			(at 166.37 73.66 0)
 			(effects
@@
 			)
 		)
-		(property "Footprint" "Resistor_SMD:R_0402_1005Metric_Pad0.72x0.64mm_HandSolder"
+		(property "Footprint" "Resistor_SMD:R_0603_1608Metric_Pad0.98x0.95mm_HandSolder"
 			(at 156.21 61.722 90)
 			(effects
@@
 			)
 		)
-		(property "DigiKey Part #" "P47DCCT-ND"
+		(property "DigiKey Part #" "311-47.0HRCT-ND"
+			(at 156.21 63.5 90)
+			(effects
+				(font
+					(size 1.27 1.27)
+				)
+				(hide yes)
+			)
+		)
+		(property "JLCPCB Part #" "C23182"
 			(at 156.21 63.5 90)
 			(effects
@@
 			)
 		)
+		(property "JLCPCB Part #" "C25744"
+			(at 143.51 123.19 0)
+			(effects
+				(font
+					(size 1.27 1.27)
+				)
+				(hide yes)
+			)
+		)
 		(pin "1"
 		)
@@
 			)
 		)
+		(property "JLCPCB Part #" ""
+			(at 69.85 40.64 0)
+			(effects
+				(font
+					(size 1.27 1.27)
+				)
+				(hide yes)
+			)
+		)
 		(pin "1"
 		)
@@
 			)
 		)
+		(property "JLCPCB Part #" "C28233"
+			(at 143.51 101.6 0)
+			(effects
+				(font
+					(size 1.27 1.27)
+				)
+				(hide yes)
+			)
+		)
 		(pin "2"
 		)
@@
 		)
 		(property "DigiKey Part #" "1276-3431-1-ND"
+			(at 134.62 149.86 0)
+			(effects
+				(font
+					(size 1.27 1.27)
+				)
+				(hide yes)
+			)
+		)
+		(property "JLCPCB Part #" "C25744"
 			(at 134.62 149.86 0)
 			(effects
@@
 			)
 		)
+		(property "JLCPCB Part #" "C28233"
+			(at 143.51 134.62 0)
+			(effects
+				(font
+					(size 1.27 1.27)
+				)
+				(hide yes)
+			)
+		)
 		(pin "2"
 		)
@@
 			)
 		)
-		(property "Footprint" "Resistor_SMD:R_0402_1005Metric_Pad0.72x0.64mm_HandSolder"
+		(property "Footprint" "Resistor_SMD:R_0603_1608Metric_Pad0.98x0.95mm_HandSolder"
 			(at 156.21 94.742 90)
 			(effects
@@
 			)
 		)
-		(property "DigiKey Part #" "P47DCCT-ND"
+		(property "DigiKey Part #" "311-47.0HRCT-ND"
+			(at 156.21 96.52 90)
+			(effects
+				(font
+					(size 1.27 1.27)
+				)
+				(hide yes)
+			)
+		)
+		(property "JLCPCB Part #" "C23182"
 			(at 156.21 96.52 90)
 			(effects
@@
 			(at 127 113.03 0)
 			(effects
+				(font
+					(size 1.27 1.27)
+				)
+				(hide yes)
+			)
+		)
+		(property "JLCPCB Part #" ""
+			(at 127 113.03 0)
+			(effects

Commit message: user save part number
Parts:
- U102, U401: JLCPCB Part # (none) -> C5605

Commit message: user save
Parts:
- removed U102, U401: 74HC14, Package_SO:SOIC-14_3.9x8.7mm_P1.27mm, symbol 74xx:74HC14
- added U11: 74HC14, Package_SO:SOIC-14_3.9x8.7mm_P1.27mm, symbol 74xx:74HC14
Connections:
- net +3V3: now also U11.14 (VCC)
- net Debouncer_Out_1: now also U11.2
- net Debouncer_Out_2: now also U11.4
- net Debouncer_Out_3: now also U11.6
- net Debouncer_Out_4: now also U11.8
- net Debouncer_Out_5: now also U11.10
- net GND: now also U11.7 (GND)
- net at R113.2: now also U11.13
- net at C106.1, R111.1, R112.2: now also U11.11
- net at C103.1, R105.1, R106.2: now also U11.3
- net at C104.1, R107.1, R108.2: now also U11.5
- net at C102.1, R102.2, R104.1: now also U11.1
- net at C105.1, R109.1, R110.2: now also U11.9
