File: Systemboard/Systemboard.kicad_pcb (KiCad board)
At the start: 2 copper layers, 192 parts, among them J1 Conn_01x60, J108 Prog BT, J2 Conn_01x02, J3 Conn_01x01, J4 Conn_01x01, Q1 MMBT5551L, Q2 MMBT5551L, Q3 MMBT5551L, Q4 MMBT5551L, Q5 MMBT5551L, U1 INA226, U10 74HC595, U101 ESP32-WROOM-32E, U103 TLV73333PDBV, U104 PCM2706CPJTR, U11 74HC14, U2 LM358, U201 TLV73333PDBV, U202 PCM5102A, U3 J104D2C12VDC.15S, U301 TLV73333PDBV, U4 J104D2C12VDC.15S, U5 LM2596S-5, U501 TPA3118D2DAPR, U6 LM2596S-3.3, U7 LM2596S-5, U8 LM2596S-ADJ, U9 LTV-817S, Y101 CSTNE12M0G55A000R0

Commit message: replace pot
Parts:
- added RV1: 10k, External_Parts:Fader 401766, F.Cu at (314.8, 265.0)
Other:
- board outline added: 53.7 x 2 mm
Changed lines of the file:
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@@
 		)
+	)
+	(footprint "External_Parts:Fader 401766"
+		(layer "F.Cu")
+		(at 314.75 265.025)
+		(property "Reference" "RV1"
+			(at 0 -0.5 0)
+			(unlocked yes)
+			(layer "F.SilkS")
+			(effects
+				(font
+					(size 1 1)
+					(thickness 0.1)
+				)
+			)
+		)
+		(property "Value" "10k"
+			(at 0 1 0)
+			(unlocked yes)
+			(layer "F.Fab")
+			(effects
+				(font
+					(size 1 1)
+					(thickness 0.15)
+				)
+			)
+		)
+		(property "Datasheet" ""
+			(at 0 0 0)
+			(unlocked yes)
+			(layer "F.Fab")
+			(hide yes)
+			(effects
+				(font
+					(size 1 1)
+					(thickness 0.15)
+				)
+			)
+		)
+		(property "Description" "Dual potentiometer"
+			(at 0 0 0)
+			(unlocked yes)
+			(layer "F.Fab")
+			(hide yes)
+			(effects
+				(font
+					(size 1 1)
+					(thickness 0.15)
+				)
+			)
+		)
+		(property "Sim.Library" "${KICAD9_SYMBOL_DIR}/Simulation_SPICE.sp"
+			(at 0 0 0)
+			(unlocked yes)
+			(layer "F.Fab")
+			(hide yes)
+			(effects
+				(font
+					(size 1 1)
+					(thickness 0.15)
+				)
+			)
+		)
+		(property "Sim.Name" "pot_dual"
+			(at 0 0 0)
+			(unlocked yes)
+			(layer "F.Fab")
+			(hide yes)
+			(effects
+				(font
+					(size 1 1)
+					(thickness 0.15)
+				)
+			)
+		)
+		(property "Sim.Device" "SUBCKT"
+			(at 0 0 0)
+			(unlocked yes)
+			(layer "F.Fab")
+			(hide yes)
+			(effects
+				(font
+					(size 1 1)
+					(thickness 0.15)
+				)
+			)
+		)
+		(property "Sim.Pins" "1=r1A 2=wA 3=r0A 4=r1B 5=wB 6=r0B"
+			(at 0 0 0)
+			(unlocked yes)
+			(layer "F.Fab")
+			(hide yes)
+			(effects
+				(font
+					(size 1 1)
+					(thickness 0.15)
+				)
+			)
+		)
+		(property "Sim.Params" "Rtot=1 wpos=0.4"
+			(at 0 0 0)
+			(unlocked yes)
+			(layer "F.Fab")
+			(hide yes)
+			(effects
+				(font
+					(size 1 1)
+					(thickness 0.15)
+				)
+			)
+		)
+		(property ki_fp_filters "Potentiometer*")
+		(sheetname "/")
+		(sheetfile "Systemboard.kicad_sch")
+		(units
+			(unit
+				(name "A")
+				(pins "1" "2" "3" "4" "5" "6")
+			)
+		)
+		(attr through_hole)
+		(duplicate_pad_numbers_are_jumpers no)
+		(fp_circle
+			(center -25.85 0)
+			(end -24.85 0)
+			(stroke
+				(width 0.05)
+				(type solid)
+			)
+			(fill no)
+			(layer "Edge.Cuts")
+		)
+		(fp_circle
+			(center 25.85 0)
+			(end 26.85 0)
+			(stroke
+				(width 0.05)
+				(type solid)
+			)
+			(fill no)
+			(layer "Edge.Cuts")
+		)
+		(fp_rect
+			(start -44 -8)
+			(end 44 8)
+			(stroke
+				(width 0.05)
+				(type solid)
+			)
+			(fill no)
+			(layer "F.CrtYd")
+		)
+		(fp_text user "${REFERENCE}"
+			(at 0 2.5 0)
+			(unlocked yes)
+			(layer "F.Fab")
+			(effects
+				(font
+					(size 1 1)
+					(thickness 0.15)
+				)
+			)
+		)
+		(pad "1" thru_hole oval
+			(at 43.75 -1.875)
+			(size 4 3)
+			(drill 1.5)
+			(layers "*.Cu" "*.Mask")
+			(remove_unused_layers no)
+			(net "/Amplifier Input Mux/AMPLIFIER_IN_L")
+			(pinfunction "1_1")
+			(pintype "passive")
+		)
+		(pad "2" thru_hole oval
+			(at -43.75 -5.625)
+			(size 4 3)
+			(drill 1.5)
+			(layers "*.Cu" "*.Mask")
+			(remove_unused_layers no)
+			(net "/Amplifier/Amplifier_In_L")
+			(pinfunction "2_2")
+			(pintype "passive")
+		)
+		(pad "3" thru_hole oval
+			(at -43.75 -1.875)
+			(size 4 3)
+			(drill 1.5)
+			(layers "*.Cu" "*.Mask")
+			(remove_unused_layers no)
+			(net "GND")
+			(pinfunction "3_3")
+			(pintype "passive")
+		)
+		(pad "4" thru_hole oval
+			(at 43.75 1.875)
+			(size 4 3)
+			(drill 1.5)
+			(layers "*.Cu" "*.Mask")
+			(remove_unused_layers no)
+			(net "/Amplifier Input Mux/AMPLIFIER_IN_R")
+			(pinfunction "4_4")
+			(pintype "passive")
+		)
+		(pad "5" thru_hole oval
+			(at -43.75 5.625)
+			(size 4 3)
+			(drill 1.5)
+			(layers "*.Cu" "*.Mask")
+			(remove_unused_layers no)
+			(net "/Amplifier/Amplifier_In_R")
+			(pinfunction "5_5")
+			(pintype "passive")
+		)
+		(pad "6" thru_hole oval
+			(at -43.75 1.875)
+			(size 4 3)
+			(drill 1.5)
+			(layers "*.Cu" "*.Mask")
+			(remove_unused_layers no)
+			(net "GND")
+			(pinfunction "6_6")
+			(pintype "passive")
+		)
+		(embedded_fonts no)
 	)
 	(footprint "Resistor_SMD:R_0402_1005Metric_Pad0.72x0.64mm_HandSolder"

Commit message: user save
Parts:
- added REF**: MountingHole_3.2mm_M3, MountingHole:MountingHole_3.2mm_M3, F.Cu at (97.0, 153.5)
- added REF**: MountingHole_3mm, MountingHole:MountingHole_3mm, F.Cu at (189.5, 77.0)
- added REF**: MountingHole_3.2mm_M3, MountingHole:MountingHole_3.2mm_M3, F.Cu at (26.0, 153.5)
- added REF**: MountingHole_3mm, MountingHole:MountingHole_3mm, F.Cu at (149.5, 77.0)
- added REF**: MountingHole_3.2mm_M3, MountingHole:MountingHole_3.2mm_M3, F.Cu at (46.5, 142.5)
- added REF**: MountingHole_3.2mm_M3, MountingHole:MountingHole_3.2mm_M3, F.Cu at (26.0, 138.5)
- added REF**: MountingHole_3.2mm_M3, MountingHole:MountingHole_3.2mm_M3, F.Cu at (76.5, 142.5)
- added REF**: MountingHole_3.2mm_M3, MountingHole:MountingHole_3.2mm_M3, F.Cu at (61.5, 142.5)
- added REF**: MountingHole_3.2mm_M3, MountingHole:MountingHole_3.2mm_M3, F.Cu at (97.0, 138.5)
- R150, R152, RV1, S1, S2: moved to B.Cu
- moved C27 444.0 mm to (30.8, 80.4), turned to 180 degrees
- moved U6 427.1 mm to (39.6, 90.8), turned to -90 degrees
- moved L5 426.6 mm to (39.6, 71.9), turned to 180 degrees
- moved R141 418.2 mm to (94.4, 30.8), turned to -90 degrees
- moved U9 413.3 mm to (101.4, 31.3), turned to 0 degrees
- moved R148 411.5 mm to (28.9, 47.6), turned to 0 degrees
- moved R147 410.8 mm to (111.5, 28.8), turned to 180 degrees
- moved R139 409.1 mm to (108.9, 31.2), turned to 90 degrees
- moved R140 408.2 mm to (110.4, 31.2), turned to -90 degrees
- moved C26 408.2 mm to (48.8, 81.9), turned to 0 degrees
- moved Q4 406.8 mm to (113.9, 30.8), turned to 90 degrees
- moved D2 405.8 mm to (50.1, 69.4), turned to 90 degrees
- moved C25 405.6 mm to (31.6, 43.1), turned to 180 degrees
- moved Q5 404.7 mm to (32.4, 48.6), turned to 0 degrees
- moved C32 404.4 mm to (119.7, 30.3), turned to 0 degrees
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Other:
- board size 53.7 x 2 mm -> 175 x 135 mm
