File: Systemboard/Systemboard.kicad_pcb (KiCad board)
At the start: 2 copper layers, 175 x 135 mm, 202 parts, among them J1 Conn_01x60, J108 Prog BT, J2 Conn_01x02, J3 Conn_01x01, J4 Conn_01x01, Q1 MMBT5551L, Q2 MMBT5551L, Q3 MMBT5551L, Q4 MMBT5551L, Q5 MMBT5551L, U1 INA226, U10 74HC595, U101 ESP32-WROOM-32E, U103 TLV73333PDBV, U104 PCM2706CPJTR, U11 74HC14, U2 LM358, U201 TLV73333PDBV, U202 PCM5102A, U3 J104D2C12VDC.15S, U301 TLV73333PDBV, U4 J104D2C12VDC.15S, U5 LM2596S-5, U501 TPA3118D2DAPR, U6 LM2596S-3.3, U7 LM2596S-5, U8 LM2596S-ADJ, U9 LTV-817S, Y101 CSTNE12M0G55A000R0

Commit message: new selector
Parts:
- removed the REF** at (97.0, 153.5)
- removed the REF** at (26.0, 153.5)
- removed the REF** at (46.5, 142.5)
- removed the REF** at (26.0, 138.5)
- removed the REF** at (76.5, 142.5)
- removed the REF** at (61.5, 142.5)
- removed the REF** at (97.0, 138.5)
- added REF**: MountingHole_2.5mm, MountingHole:MountingHole_2.5mm, F.Cu at (84.5, 153.5)
- added REF**: MountingHole_2.5mm, MountingHole:MountingHole_2.5mm, F.Cu at (114.5, 153.5)
- added REF**: microswitch, External_Parts:microswitch, F.Cu at (54.5, 132.0)
- added REF**: MountingHole_2.5mm, MountingHole:MountingHole_2.5mm, F.Cu at (129.5, 153.5)
- added REF**: MountingHole_2.5mm, MountingHole:MountingHole_2.5mm, F.Cu at (54.5, 153.5)
- added REF**: MountingHole_2.5mm, MountingHole:MountingHole_2.5mm, F.Cu at (99.5, 153.5)
- added REF**: MountingHole_2.5mm, MountingHole:MountingHole_2.5mm, F.Cu at (24.5, 153.5)
- added REF**: MountingHole_2.5mm, MountingHole:MountingHole_2.5mm, F.Cu at (69.5, 153.5)
- added REF**: MountingHole_2.5mm, MountingHole:MountingHole_2.5mm, F.Cu at (39.5, 153.5)
- R150, R152: moved to F.Cu
- S1, S2: footprint External_Parts:SS0750301F040P1A -> External_Parts:microswitch; moved to F.Cu
- moved S2 61.4 mm to (94.5, 132.0)
- moved R152 61.2 mm to (88.4, 116.0)
- moved R150 39.1 mm to (78.0, 116.5), turned to 0 degrees
- moved C30 32.2 mm to (27.7, 86.4), turned to -90 degrees
- moved C29 30.2 mm to (43.7, 90.3), turned to 90 degrees
- moved L7 29.5 mm to (36.2, 88.1), turned to 90 degrees
- moved C119 28.9 mm to (133.4, 60.1)
- moved U10 28.9 mm to (140.0, 63.5)
- moved C27 28.1 mm to (49.1, 59.0), turned to 90 degrees
- moved D3 26.2 mm to (51.2, 110.6), turned to 0 degrees
- moved L6 25.9 mm to (48.7, 99.6), turned to 90 degrees
- moved U6 23.0 mm to (38.7, 67.8), turned to 180 degrees
- moved R103 22.9 mm to (91.9, 61.8)
- moved C201 22.9 mm to (102.5, 63.0)
- moved C202 22.9 mm to (101.0, 57.5)
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
Commit message: mechanical adjustments
Parts:
- removed the REF** at (129.5, 153.5)
- added REF**: MountingHole_4.3mm_M4, MountingHole:MountingHole_4.3mm_M4, F.Cu at (52.0, 130.0)
- added REF**: MountingHole_4.3mm_M4, MountingHole:MountingHole_4.3mm_M4, F.Cu at (165.0, 37.0)
- added REF**: MountingHole_4.3mm_M4, MountingHole:MountingHole_4.3mm_M4, F.Cu at (111.0, 32.0)
- added REF**: MountingHole_4.3mm_M4, MountingHole:MountingHole_4.3mm_M4, F.Cu at (186.0, 114.0)
- REF**, S1, S2: moved to B.Cu
- moved R152 20.2 mm to (108.6, 116.5), turned to 90 degrees
- moved D7 14.6 mm to (198.0, 114.5)
- moved Q1 14.6 mm to (205.0, 113.5)
- moved R134 14.6 mm to (205.0, 116.5)
- moved U3 14.6 mm to (201.8, 109.9)
- moved C101 14.1 mm to (130.5, 84.3)
- moved C106 14.1 mm to (139.4, 67.5)
- moved C401 14.1 mm to (137.1, 63.4)
- moved D2 14.1 mm to (74.1, 76.3)
- moved L5 14.1 mm to (71.6, 65.8)
- moved C1 14.1 mm to (172.0, 76.5)
- moved C10 14.1 mm to (195.0, 47.5)
- moved C102 14.1 mm to (127.4, 63.7)
- moved C103 14.1 mm to (127.4, 67.5)
- moved C104 14.1 mm to (127.4, 71.3)
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
Commit message: update
Parts:
- added REF**: MountingHole_4.3mm_M4, MountingHole:MountingHole_4.3mm_M4, F.Cu at (64.0, 59.0)
- moved C101 79.8 mm to (55.9, 112.7), turned to -90 degrees
- moved R117 77.2 mm to (55.1, 110.4), turned to 180 degrees
- moved R101 73.8 mm to (55.9, 108.1), turned to -90 degrees
- moved R151 72.6 mm to (57.7, 108.0), turned to -90 degrees
- moved R153 71.6 mm to (59.4, 108.0), turned to -90 degrees
- moved C216 70.4 mm to (54.8, 104.9), turned to 180 degrees
- moved C217 67.5 mm to (54.9, 102.6), turned to 0 degrees
- moved C208 67.1 mm to (90.0, 111.9), turned to 180 degrees
- moved U201 66.9 mm to (85.0, 113.4), turned to 0 degrees
- moved C204 65.8 mm to (97.0, 107.4), turned to -90 degrees
- moved C205 63.8 mm to (90.0, 109.4), turned to 180 degrees
- moved R201 62.7 mm to (96.9, 104.9), turned to 0 degrees
- moved C201 62.5 mm to (79.5, 111.4), turned to 90 degrees
- moved C212 62.4 mm to (94.0, 106.4), turned to 90 degrees
- moved C202 62.1 mm to (85.0, 109.9), turned to 180 degrees
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Other:
- outline, holes or cut-outs redrawn

Commit message: update
Parts:
- removed the REF** at (123.5, 151.5)
- removed the REF** at (47.0, 130.0)
- removed the REF** at (126.5, 59.0)
- removed the REF** at (146.0, 146.0)
- added REF**: MountingHole_2.7mm_M2.5, MountingHole:MountingHole_2.7mm_M2.5, F.Cu at (44.2, 135.6)
- added REF**: MountingHole_2.7mm_M2.5, MountingHole:MountingHole_2.7mm_M2.5, F.Cu at (207.2, 139.6)
- moved REF** 51.7 mm to (208.2, 55.6)
- moved R148 42.4 mm to (70.0, 22.9), turned to -90 degrees
- moved C25 41.0 mm to (74.5, 25.6), turned to 90 degrees
- moved L4 39.7 mm to (84.0, 34.1), turned to 90 degrees
- moved Q5 37.2 mm to (69.0, 26.4), turned to -90 degrees
- moved D1 35.8 mm to (86.5, 44.9), turned to 0 degrees
- moved R149 34.9 mm to (65.4, 27.4), turned to 180 degrees
- moved L5 33.4 mm to (90.3, 66.4)
- moved U6 33.4 mm to (109.2, 66.4)
- moved C26 33.4 mm to (100.3, 57.3)
- moved D2 33.4 mm to (87.8, 55.9)
- moved C27 33.4 mm to (98.8, 75.2)
- moved C28 33.1 mm to (120.4, 98.6)
- moved C29 33.1 mm to (126.0, 79.7)
- moved C30 33.1 mm to (110.0, 75.8)
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Other:
- outline, holes or cut-outs redrawn

Commit message: update
Parts:
- moved R102 10.1 mm to (176.8, 107.0)
- moved R106 10.1 mm to (179.3, 107.0)
- moved R108 10.1 mm to (182.9, 107.0)
- moved R110 10.1 mm to (184.9, 107.0)
- moved R112 10.1 mm to (186.9, 107.0)
- moved J1 10.1 mm to (190.5, 117.5)
- moved R137 7.83 mm to (201.0, 109.5)
- moved R138 7.60 mm to (199.0, 109.5)
- moved D7 6.73 mm to (208.0, 107.0)
- moved Q1 6.73 mm to (215.0, 106.0)
- moved R134 6.73 mm to (215.0, 109.0)
- moved U3 6.73 mm to (211.8, 102.4)
- moved REF** 4.26 mm to (48.2, 137.1)
- moved REF** 4.03 mm to (211.2, 140.1)
- moved C217 4.03 mm to (67.9, 102.1)
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Other:
- outline, holes or cut-outs redrawn
