File: Systemboard/Systemboard.kicad_pcb (KiCad board)
At the start: 2 copper layers, 175 x 135 mm, 206 parts, among them J1 Conn_01x60, J108 Prog BT, J2 Conn_01x02, J3 Conn_01x01, J4 Conn_01x01, Q1 MMBT5551L, Q2 MMBT5551L, Q3 MMBT5551L, Q4 MMBT5551L, Q5 MMBT5551L, U1 INA226, U10 74HC595, U101 ESP32-WROOM-32E, U103 TLV73333PDBV, U104 PCM2706CPJTR, U11 74HC14, U2 LM358, U201 TLV73333PDBV, U202 PCM5102A, U3 J104D2C12VDC.15S, U301 TLV73333PDBV, U4 J104D2C12VDC.15S, U5 LM2596S-5, U501 TPA3118D2DAPR, U6 LM2596S-3.3, U7 LM2596S-5, U8 LM2596S-ADJ, U9 LTV-817S, Y101 CSTNE12M0G55A000R0

Commit message: via stitching
Routing:
- net GND: vias 74 -> 406

Commit message: Update Systemboard.kicad_pcb
Routing:
- net +12V: track 37.7 -> 308.4 mm, vias 0 -> 11
- net +5V: track 21.8 -> 290.6 mm, vias 0 -> 3
- net +3V3: track 20.9 -> 278.7 mm, vias 0 -> 7
- net /USB_DAC_CABLE_DETECT_B: track 0.00 -> 170.2 mm, vias 0 -> 4
- net /Dimmable_V+: track 7.59 -> 146.3 mm, vias 0 -> 2
- net /USB_DAC_CABLE_DETECT_A: track 0.00 -> 136.4 mm, vias 0 -> 4
- net /Illumination: track 0.00 -> 133.2 mm, vias 0 -> 2
- net Net-(U1-Vbus): track 8.79 -> 140.2 mm, vias 0 -> 7
- net /Amplifier Input Mux/BT_DAC_R: track 0.00 -> 124.9 mm, vias 0 -> 4
- net /Amplifier/Amplifier_In_L: track 0.00 -> 115.1 mm, vias 0 -> 1
- net /~{AMP_FAIL}: track 1.50 -> 115.1 mm, vias 0 -> 4
- net /Configurator/+5V_On: track 0.00 -> 112.5 mm, vias 0 -> 2
- net /Amplifier Input Mux/BT_DAC_L: track 0.00 -> 111.7 mm, vias 0 -> 3
- net /Amplifier Input Mux/~{BT}/USB_SELECT: track 0.00 -> 90.7 mm, vias 0 -> 2
- net /Amplifier/Amplifier_In_R: track 0.00 -> 87.1 mm, vias 0 -> 1
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- added copper zone on B.Cu, net GND
- added copper zone on In1.Cu, net GND
- added copper zone on In2.Cu, net GND
Other:
- copper layers 2 -> 4

Commit message: user save
Routing:
- net /Display_SR: track 0.00 -> 177.2 mm, vias 0 -> 4
- net /Display_SRCL: track 0.00 -> 173.2 mm, vias 0 -> 4
- net /Display_RCL: track 0.00 -> 168.5 mm, vias 0 -> 4
- net /CHARGER_SHUNT_SDA: track 0.00 -> 142.3 mm, vias 0 -> 6
- net /CHARGER_SHUNT_SCL: track 0.00 -> 116.3 mm, vias 0 -> 2
- net /CHARGER_VBUS: track 0.00 -> 104.5 mm, vias 0 -> 6
- net /BTN_1_COM_B: track 0.00 -> 87.8 mm, vias 0 -> 4
- net +12V: track 308.4 -> 389.4 mm, vias 11 -> 12
- net /DAC_CC1: track 2.48 -> 80.9 mm, vias 0 -> 2
- net /BTN_5_NO_B: track 0.00 -> 63.5 mm, vias 0 -> 4
- net /BTN_4_NO_B: track 0.00 -> 56.2 mm, vias 0 -> 6
- net /DAC_VBUS: track 3.14 -> 58.8 mm
- net +3V3: track 278.7 -> 333.2 mm, vias 7 -> 9
- net /DAC_CC2: track 2.47 -> 51.9 mm, vias 0 -> 4
- net /BTN_3_NO_B: track 0.00 -> 45.3 mm, vias 0 -> 2
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Other:
- board text added: "Acc+"
- board text added: "B+"
- board text added: "GND"
- board text added: "Ill."
- board text added: "R+ R- L+ L-"

Commit message: release candidate
Parts:
- added G1: LOGO, LOGO, F.Cu at (144.0, 133.8)
- added G2: LOGO, LOGO, F.Cu at (162.2, 64.6)
Routing:
- net /USB_DAC_CABLE_DETECT_B: track 173.6 -> 174.2 mm
